File: BreathalyzerPCB.kicad_sch (KiCad schematic)
At the start: 9 parts

Commit message: v1.1
Parts:
- removed U?: MAX874, symbol Reference_Voltage:MAX874
- added BT102: 3V, symbol Device:Battery
- added R101, R103: 220, symbol Device:R_Small_US
- added U101: MAX6105, Package_TO_SOT_SMD:SOT-23, symbol Reference_Voltage:MAX6105
- BT101: renamed from BT?; value Battery -> 3V
- gave numbers to parts that had none: 7
Connections:
- net at D102.1 (K): now also R104.1
- net at D102.2 (A): now also U102.20 (D2)
- net at BT101.1 (+): now also SW101.1 (A)
- net at BT101.2 (-): now also BT102.1 (+)
- net GND: now reaches R104.2
- net GND: now also D101.1 (RK), D101.2 (GK), D101.3 (BK), U102.14 (GND), U102.19 (GND), U103.5, BT102.2 (-), U101.3 (GND)
- net VCC: now reaches U102.4 (A0/DAC0)
- net VCC: now also U103.2, U101.2 (OUT)
- net at U102.5 (A1): now also R101.1
- net at U102.6 (A2): now also R102.1
- net at U102.7 (A3): now also R103.1
- net at U102.8 (A4/SDA): now also U103.1, U103.3
- net at D101.4 (BA): now also R103.2
- net at D101.5 (GA): now also R102.2
- net at D101.6 (RA): now also R101.2
- net at SW101.2 (B): now also U101.1 (IN)
- no-connect marks 0 -> 22
Other:
- note added: "Analog Out"
- moved on the sheet: BT101, D101, D102, R102, R104, SW101, U102, U103

Commit message: v2.1.0
Parts:
- added F?: Fuse, symbol Device:Fuse
- added H101, H102, H103, H104: MountingHole, MountingHole:MountingHole_3.2mm_M3, symbol Mechanical:MountingHole
- added J101: Power Switch, Connector_PinHeader_2.54mm:PinHeader_1x02_P2.54mm_Vertical, symbol Connector:Conn_01x02_Male
- added J102: Battery, Connector_PinHeader_2.54mm:PinHeader_1x02_P2.54mm_Vertical, symbol Connector:Conn_01x02_Male
- added J103: Conn_01x03_Male, Connector_PinHeader_2.54mm:PinHeader_1x03_P2.54mm_Vertical, symbol Connector:Conn_01x03_Male
- added J104: Read LED, Connector_PinHeader_2.54mm:PinHeader_1x02_P2.54mm_Vertical, symbol Connector:Conn_01x02_Male
- added J105: MQ3, Connector_PinHeader_2.54mm:PinHeader_1x03_P2.54mm_Vertical, symbol Connector:Conn_01x03_Male
- added TP101: GND, TestPoint:TestPoint_Pad_D4.0mm, symbol Connector:TestPoint_Flag
- added TP102: AnalogMQ3, TestPoint:TestPoint_Pad_D4.0mm, symbol Connector:TestPoint_Flag
- added TP103: VCC, TestPoint:TestPoint_Pad_D4.0mm, symbol Connector:TestPoint_Flag
- R101, R102, R103, R104: footprint (none) -> Resistor_THT:R_Axial_DIN0309_L9.0mm_D3.2mm_P12.70mm_Horizontal
- U102: footprint MODULE_ABX00030 -> Connector_PinSocket_2.54mm:PinSocket_2x14_P2.54mm_Vertical
- U103: value SEN-08880 -> MQ3
Connections:
- net GND: now also U103.2, J102.1 (Pin_1), J105.1 (Pin_1), TP101.1; no longer U103.5
- net VCC: now also U102.11 (A7), U102.15 (VIN), U103.5, J105.3 (Pin_3), TP103.1; no longer U102.4 (A0/DAC0), U103.2
- net at D102.1 (K), R104.1: now also J104.1 (Pin_1)
- net ReadLED: now reaches D102.2 (A), U102.20 (D2)
- net ReadLED: now also J104.2 (Pin_2)
- net Switch: now reaches SW101.2 (B), U101.1 (IN)
- net Switch: now also J101.1 (Pin_1)
- net +6V: now reaches BT101.1 (+), SW101.1 (A)
- net +6V: now also J101.2 (Pin_2), J102.2 (Pin_2)
- net BattLED1: now reaches R101.1, U102.5 (A1)
- net BattLED1: now also J103.3 (Pin_3)
- net BattLED2: now reaches R102.1, U102.6 (A2)
- net BattLED2: now also J103.2 (Pin_2)
- net BattLED3: now reaches R103.1, U102.7 (A3)
- net BattLED3: now also J103.1 (Pin_1)
- net MQ3Analog: now reaches U102.8 (A4/SDA), U103.1, U103.3
- net MQ3Analog: now also J105.2 (Pin_2), TP102.1
- no-connect marks 22 -> 21
Other:
- moved on the sheet: BT102, D101, D102, R101, R102, R103, R104, U101, U102, U103

Commit message: v3.0.0
Parts:
- F101: renamed from F?; footprint (none) -> Fuse:Fuse_0805_2012Metric_Pad1.15x1.40mm_HandSolder
- J103: value Conn_01x03_Male -> RGBConn
- U102: footprint Connector_PinSocket_2.54mm:PinSocket_2x14_P2.54mm_Vertical -> ABX00030:MODULE_ABX00030
Connections:
- net +6V: now also F101.1, F101.2
- net BattLED1: now also D101.1 (RK), D101.6 (RA), R101.2; no longer R101.1
- net BattLED2: now also D101.2 (GK), D101.5 (GA)
- net BattLED3: now also D101.3 (BK), D101.4 (BA)
- net GND: now also R101.1, R102.2, R103.2; no longer D101.1 (RK), D101.2 (GK), D101.3 (BK)
Other:
- moved on the sheet: BT101, BT102, D101, F101, R101, R102, R103

Commit message: v4.1.0
Parts:
- removed H104: MountingHole, MountingHole:MountingHole_3.2mm_M3, symbol Mechanical:MountingHole
- added NT101: USB_Volt, NetTie:NetTie-2_THT_Pad1.0mm, symbol Device:NetTie_2
- added NT102: USB_GND, NetTie:NetTie-2_THT_Pad1.0mm, symbol Device:NetTie_2
- added P101: USBC, 105450-0101:MOLEX_105450-0101, symbol Connector:USB_C_Plug
Connections:
- net +6V: now also NT101.2
- net GND: now also NT102.2
- new net USBC: NT101.1, P101.A4 (VBUS), P101.A9 (VBUS), P101.B4 (VBUS), P101.B9 (VBUS)
- new net USBC-GND: NT102.1, P101.A1 (GND), P101.A12 (GND), P101.B1 (GND), P101.B12 (GND)
- no-connect marks 21 -> 36
Other:
- moved on the sheet: BT101, BT102, F101, J102, TP101, TP102, TP103, U101, U102

Commit message: v4.4.0
Parts:
- removed NT101: USB_Volt, NetTie:NetTie-2_THT_Pad1.0mm, symbol Device:NetTie_2
- removed NT102: USB_GND, NetTie:NetTie-2_THT_Pad1.0mm, symbol Device:NetTie_2
- removed P101: USBC, 105450-0101:MOLEX_105450-0101, symbol Connector:USB_C_Plug
- added J106: Barrel_Jack_Switch, Connector_BarrelJack:BarrelJack_Wuerth_6941xx301002, symbol Connector:Barrel_Jack_Switch
- added TP104: BattLED1Test, TestPoint:TestPoint_Pad_D4.0mm, symbol Connector:TestPoint_Flag
- added TP105: BattLED2Test, TestPoint:TestPoint_Pad_D4.0mm, symbol Connector:TestPoint_Flag
- added TP106: BattLED3Test, TestPoint:TestPoint_Pad_D4.0mm, symbol Connector:TestPoint_Flag
Connections:
- net +6V: now also J106.1
- net BattLED1: now also TP104.1
- net BattLED2: now also TP105.1
- net BattLED3: now also TP106.1
- net GND: now also J106.2, J106.3
- no-connect marks 36 -> 21
